File: owl_v1.kicad_sch (KiCad schematic)
At the start: 14 parts, among them SW1 SW_SPDT, U1 STM32F103C8T6, Y1 8MHz, Y2 32k768

Commit message: [refactor] Change the CAN Tx and Rx from global to hierarchical label
Other:
- sheet CAN Transceiver ports: added CAN_RX, CAN_TX; removed none
Changed lines of the file:
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@@
 	(wire
 		(pts
+			(xy 57.15 173.99) (xy 63.5 173.99)
+		)
+		(stroke
+			(width 0)
+			(type default)
+		)
+	)
+	(wire
+		(pts
 			(xy 34.29 63.5) (xy 36.83 63.5)
 		)
@@
 	(wire
 		(pts
+			(xy 57.15 170.18) (xy 63.5 170.18)
+		)
+		(stroke
+			(width 0)
+			(type default)
+		)
+	)
+	(wire
+		(pts
 			(xy 57.15 148.59) (xy 60.96 148.59)
 		)
@@
 		)
 	)
+	(global_label "CAN_RX"
+		(shape input)
+		(at 63.5 170.18 0)
+		(fields_autoplaced yes)
+		(effects
+			(font
+				(size 1.27 1.27)
+			)
+			(justify left)
+		)
+		(property "Intersheetrefs" "${INTERSHEET_REFS}"
+			(at 73.6214 170.18 0)
+			(hide yes)
+			(show_name no)
+			(do_not_autoplace no)
+			(effects
+				(font
+					(size 1.27 1.27)
+				)
+				(justify left)
+			)
+		)
+	)
 	(global_label "LSE_OSC_OUT"
 		(shape input)
@@
 		)
 	)
+	(global_label "CAN_TX"
+		(shape input)
+		(at 63.5 173.99 0)
+		(fields_autoplaced yes)
+		(effects
+			(font
+				(size 1.27 1.27)
+			)
+			(justify left)
+		)
+		(property "Intersheetrefs" "${INTERSHEET_REFS}"
+			(at 73.319 173.99 0)
+			(hide yes)
+			(show_name no)
+			(do_not_autoplace no)
+			(effects
+				(font
+					(size 1.27 1.27)
+				)
+				(justify left)
+			)
+		)
+	)
 	(symbol
 		(lib_id "Device:C")
@@
 	(sheet
 		(at 19.05 165.1)
-		(size 38.1 20.32)
+		(size 38.1 13.97)
 		(exclude_from_sim no)
 		(in_bom yes)
@@
 		)
 		(property "Sheetfile" "can_controller.kicad_sch"
-			(at 19.05 186.0046 0)
+			(at 19.05 179.6546 0)
 			(hide yes)
 			(show_name no)
@@
 			)
 		)
+		(pin "CAN_RX" input
+			(at 57.15 170.18 0)
+			(effects
+				(font
+					(size 1.27 1.27)
+				)
+				(justify right)
+			)
+		)
+		(pin "CAN_TX" input
+			(at 57.15 173.99 0)
+			(effects
+				(font
+					(size 1.27 1.27)
+				)
+				(justify right)
+			)
+		)
