File: untitled.kicad_sch (KiCad schematic)
At the start: 1 part, among them J1 USB_C_Receptacle_USB2.0_14P

Commit message: [feat] Routing for FT230X USB-UART
Parts:
- removed J1: USB_C_Receptacle_USB2.0_14P, symbol Connector:USB_C_Receptacle_USB2.0_14P
Connections:
- no-connect marks 3 -> 0
