File: usb_to_uart.kicad_sch (KiCad schematic)
At the start: 6 parts, among them U3 FT230XS

Commit message: [feat] Add CAN transceiver SN65VHD230
Also ran ERC checks and add some exclusion ERC for the FT230XS due to
3V3OUT being an input pin rather than output pin
Other:
- note added: "3V3OUT is an input pin since the VCC for the FT230XS is 3.3V"
Changed lines of the file:
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@@
 	(generator_version "10.0")
 	(paper "A4")
+	(rectangle
+		(start 120.65 63.5)
+		(end 154.94 69.85)
+		(stroke
+			(width 0)
+			(type default)
+		)
+		(fill
+			(type none)
+		)
+	)
+	(text "3V3OUT is an input pin since\nthe VCC for the FT230XS is 3.3V"
+		(exclude_from_sim no)
+		(at 137.922 66.802 0)
+		(effects
+			(font
+				(size 1.27 1.27)
+			)
+		)
+	)
 	(junction
 		(at 128.27 91.44)

Commit message: [feat] Integrate MicroSD Card into the board with SPI2
Parts:
- C11, C12, C13: footprint (none) -> Capacitor_SMD:C_0603_1608Metric
- R4, R5: footprint (none) -> Resistor_SMD:R_0603_1608Metric
Changed lines of the file:
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@@
 			)
 		)
-		(property "Footprint" ""
+		(property "Footprint" "Capacitor_SMD:C_0603_1608Metric"
 			(at 118.11 96.52 0)
 			(hide yes)
@@
 			)
 		)
-		(property "Footprint" ""
+		(property "Footprint" "Resistor_SMD:R_0603_1608Metric"
 			(at 129.54 90.678 90)
 			(hide yes)
@@
 			)
 		)
-		(property "Footprint" ""
+		(property "Footprint" "Capacitor_SMD:C_0603_1608Metric"
 			(at 128.27 97.79 0)
 			(hide yes)
@@
 			)
 		)
-		(property "Footprint" ""
+		(property "Footprint" "Resistor_SMD:R_0603_1608Metric"
 			(at 135.89 93.218 90)
 			(hide yes)
@@
 			)
 		)
-		(property "Footprint" ""
+		(property "Footprint" "Capacitor_SMD:C_0603_1608Metric"
 			(at 163.83 72.39 0)
 			(hide yes)

Commit message: [feat] Add OLED I2C breakout for display, Add general purpose GPIOs
Other:
- note added: "Please refer FT230X datasheet for more info"
Changed lines of the file:
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@@
 	(paper "A4")
 	(rectangle
-		(start 120.65 63.5)
-		(end 154.94 69.85)
+		(start 134.112 51.816)
+		(end 179.832 62.738)
 		(stroke
 			(width 0)
@@
 		)
 	)
+	(text "Please refer FT230X datasheet for more info"
+		(exclude_from_sim no)
+		(at 157.48 59.69 0)
+		(effects
+			(font
+				(size 1.27 1.27)
+			)
+		)
+	)
 	(text "3V3OUT is an input pin since\nthe VCC for the FT230XS is 3.3V"
 		(exclude_from_sim no)
-		(at 137.922 66.802 0)
+		(at 156.972 55.118 0)
 		(effects
 			(font

Commit message: [feat] Integrate external battery
Parts:
- C11, C12: value 47p -> 47pF
- C13: value 100n -> 100nF
Changed lines of the file:
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@@
 			)
 		)
-		(property "Value" "47p"
+		(property "Value" "47pF"
 			(at 111.506 98.298 0)
 			(show_name no)
@@
 			)
 		)
-		(property "Value" "47p"
+		(property "Value" "47pF"
 			(at 121.92 98.552 0)
 			(show_name no)
@@
 			)
 		)
-		(property "Value" "100n"
+		(property "Value" "100nF"
 			(at 161.798 69.342 90)
 			(show_name no)

Commit message: [feat] Initial routing for the owl PCB
Parts:
- U3: private KLC_S4.2_3V3OUT -> (none)
Changed lines of the file:
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@@
-			)
-		)
-		(property private "KLC_S4.2_VCC" "This is not a power converter chip"
-			(at 157.48 125.73 0)
-			(hide yes)
-			(show_name yes)
-			(do_not_autoplace no)
-			(effects
-				(font
-					(size 1.27 1.27)
-				)
-			)
-		)
-		(property private "KLC_S4.2_3V3OUT" "This is not a power converter chip"
-			(at 157.48 128.27 0)
-			(hide yes)
-			(show_name yes)
-			(do_not_autoplace no)
-			(effects
-				(font
-					(size 1.27 1.27)
-				)
 			)
 		)

Commit message: [feat] Routing for FT230X USB-UART
Other:
- note added: "FT230X Datasheet"
- note added: "It is worth noting that the FT230X functions as a full speed USB 2.0 device (12Mb/s) as opposed to High Speed device (480Mb/s). Hence, it is not as important to match USB 2.0 impedance for the differential pairs. Although, it does not hurt to do so. Source: FT230X Datasheet, p. 29, Sec. 8.1, see USB Version description"
Changed lines of the file:
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@@
+		)
+	)
+	(rectangle
+		(start 21.59 85.09)
+		(end 97.79 104.14)
+		(stroke
+			(width 0)
+			(type default)
+		)
+		(fill
+			(type none)
 		)
 	)
@@
 		(exclude_from_sim no)
 		(at 156.972 55.118 0)
+		(effects
+			(font
+				(size 1.27 1.27)
+			)
+		)
+	)
+	(text "FT230X Datasheet"
+		(exclude_from_sim no)
+		(at 56.388 101.6 0)
+		(effects
+			(font
+				(size 1.27 1.27)
+			)
+			(href "https://www.farnell.com/datasheets/4499129.pdf")
+		)
+	)
+	(text "It is worth noting that the FT230X functions as a full speed USB 2.0\ndevice (12Mb/s) as opposed to High Speed device (480Mb/s). Hence, it is\nnot as important to match USB 2.0 impedance for the differential pairs.\nAlthough, it does not hurt to do so.\n\nSource: FT230X Datasheet, p. 29, Sec. 8.1, see USB Version description"
+		(exclude_from_sim no)
+		(at 59.436 92.456 0)
 		(effects
 			(font
@@
 		)
 	)
+	(group ""
+		(members "b2df9c03-77f2-4543-a6d9-2834f224cb40" "e00c9461-075a-43c8-88b8-25b5ec81dd4f"
+			"f9ee1db5-db00-47a5-b543-992e1efec44c"
+		)
+	)
